File: OLEDHAT.sch (EAGLE design)
At the start: 18 parts, among them IC1 MCP23017SO, J1 M40-SOCKET-BELOW, J4 DC IN

Commit message: Final routing, plus ERC and DRC for v1.0 release
Other:
- note added: "128x64 OLED Display"
- note removed: "Prototyping Area"
Changed lines of the file:
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@@
 <?xml version="1.0" encoding="utf-8"?>
 <!DOCTYPE eagle SYSTEM "eagle.dtd">
-<eagle version="9.4.2">
+<eagle version="9.5.0">
 <drawing>
 <settings>
@@
 <wire x1="119.38" y1="104.14" x2="187.96" y2="104.14" width="0.3048" layer="97" style="longdash"/>
 <wire x1="119.38" y1="104.14" x2="119.38" y2="147.32" width="0.3048" layer="97" style="longdash"/>
-<text x="124.46" y="176.53" size="1.778" layer="94">Prototyping Area</text>
+<text x="124.46" y="176.53" size="1.778" layer="94">128x64 OLED Display</text>
 <frame x1="0" y1="0" x2="248.92" y2="185.42" columns="8" rows="5" layer="94"/>
 <wire x1="119.38" y1="147.32" x2="119.38" y2="181.61" width="0.3048" layer="97" style="longdash"/>
